File: SCHEME/board.kicad_pcb (KiCad board)
At the start: 2 copper layers, 105 x 45 mm, 40 parts, among them J1 PINHD_2x4_Male, J2 PINHD_1x2_Male, J3 PINHD_1x3_Male, J4 PINHD_1x6_Male, J5 PINHD_1x6_Male, X1 Bus_ISA_8bit, X2 PINHD_1x7_Male, X3 USB_A_Stacked

Commit message: Updated board: 1. Reduced ISA slot; 2. Changed beads from 0805 to 1206; 3. General trace improvements.
Parts:
- C1, C16, C2: value 10uF_16V -> 10u
- C10, C11, C12, C13, C14, C15, C3, C9: value C_0805 -> 0.1
- C4, C5, C6, C7: value C_0805 -> 220p
- C8: value 10uF_16V -> 33u
- DD3: value EPM3064ATC44-10 -> EPM3064ATC44
- F2: value Polyfuse_3A_15V -> 500mA
- FB1, FB2, FB3, FB4: value FerriteBead -> ~; footprint Inductor_SMD:L_0805_2012Metric -> Inductor_SMD:L_1206_3216Metric_Pad1.22x1.90mm_HandSolder
- R1, R2, R3, R4: value R_0805 -> 4.7k
- R5: value R_0805 -> 560
- moved R5 15.4 mm to (170.8, 101.2)
- moved C10 2.80 mm to (163.2, 87.4)
- moved C9 2.63 mm to (166.2, 87.4)
- moved C14 1.52 mm to (129.4, 101.8)
- moved FB4 1.35 mm to (183.7, 97.8)
- moved C3 1.34 mm to (148.4, 97.5)
- moved C13 1.33 mm to (139.1, 108.2)
- moved FB1 0.95 mm to (183.7, 87.4)
- moved C15 0.90 mm to (138.4, 88.4)
- moved FB3 0.75 mm to (183.7, 94.4)
- moved FB2 0.45 mm to (183.7, 90.8)
- renumbered D1 to VD1
Routing:
- net Net-(VD1-K): track 6.26 -> 18.6 mm, vias 0 -> 2
- net /LED: track 57.6 -> 48.9 mm, vias 3 -> 0
- net /IRQ2: track 75.3 -> 68.4 mm, vias 2 -> 4
- net /IRQ4: track 37.7 -> 31.9 mm
- net +5VL: track 96.7 -> 101.5 mm, vias 3 -> 1
- net +5V: track 45.3 -> 50.0 mm, vias 1 -> 2
- net /USB_D1+: track 39.1 -> 43.7 mm
- net Net-(X3-D1+): track 18.2 -> 22.7 mm
- net +3.3V: track 107.8 -> 104.7 mm, vias 3 -> 6
- net /RTS2: track 62.4 -> 59.4 mm
- net /V3MCU: track 6.25 -> 3.34 mm
- net /IRQ3: track 34.6 -> 32.0 mm
- net /TxD: track 46.0 -> 43.6 mm
- net /CMS1: track 68.0 -> 66.1 mm
- net /USB_D2-: track 21.1 -> 22.9 mm
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Other:
- board size 105 x 45 mm -> 105 x 44.9 mm
- board text added: "COM PORT MOUSE EMULATOR"
- board text added: "LM1117-3.3"
- board text added: "https://github.com/Yftul/usb-mouse-2-isa"
- board text removed: "LM1117DT-3.3"
